File: HybridRocket2017_opening.kicad_pcb (KiCad board)
At the start: 2 copper layers, 80 x 60 mm, 48 parts, among them J1 RS485, P1 3VPWR, P2 Switch, P3 SWD, P4 Debug, P5 FlightPIN, P6 9VPWR, P7 BUZZ, P8 Valve, U1 STM32F4xxRx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

Commit message: 製作中にコミットするの忘れてた
Parts:
- moved U2 1.11 mm to (79.0, 69.0)
Routing:
- net GND: track 656.4 -> 627.9 mm, vias 96 -> 100
- net +3V3: track 122.8 -> 120.8 mm
- net /TWE_MCUTX: track 16.9 -> 17.8 mm
